File: PSU.kicad_sch (KiCad schematic)
At the start: 19 parts, among them J1 USB_C_Receptacle_USB2.0_16P, U2 LM1117DT-ADJ

Commit message: Fixing git
Parts:
- C10: value C -> .1u
- C15: renamed from C11; value C_Polarized -> 4.7u
- C9: value C -> .01u
- F1: value Polyfuse -> 500mA
- FB1: value FerriteBead -> 120
- R10: value R -> 70
- R7: value R -> 5100
- R8: value R -> 5.1k
- R9: value R -> 155
Connections:
- no-connect marks 0 -> 3
Other:
- note added: "GLOBAL LABELS"
Changed lines of the file:
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@@
   (junction (at 105.41 157.48) (diameter 0) (color 0 0 0 0)
   )
-  (junction (at 118.11 157.48) (diameter 0) (color 0 0 0 0)
-  )
   (junction (at 104.14 85.09) (diameter 0) (color 0 0 0 0)
   )
   (junction (at 81.28 85.09) (diameter 0) (color 0 0 0 0)
   )
+  (no_connect (at 193.04 74.93))
+  (no_connect (at 193.04 72.39))
+  (no_connect (at 170.18 82.55))
   (wire (pts (xy 90.17 157.48) (xy 105.41 157.48))
     (stroke (width 0) (type default))
@@
     (stroke (width 0) (type default))
   )
+  (bus (pts (xy 208.28 144.78) (xy 220.98 144.78))
+    (stroke (width 0) (type default))
+  )
   (wire (pts (xy 104.14 85.09) (xy 118.11 85.09))
     (stroke (width 0) (type default))
@@
     (stroke (width 0) (type default))
   )
+  (wire (pts (xy 92.71 92.71) (xy 92.71 96.52))
+    (stroke (width 0) (type default))
+  )
+  (wire (pts (xy 125.73 157.48) (xy 137.16 157.48))
+    (stroke (width 0) (type default))
+  )
+  (wire (pts (xy 118.11 101.6) (xy 118.11 110.49))
+    (stroke (width 0) (type default))
+  )
+  (wire (pts (xy 236.22 49.53) (xy 236.22 54.61))
+    (stroke (width 0) (type default))
+  )
+  (wire (pts (xy 193.04 49.53) (xy 236.22 49.53))
+    (stroke (width 0) (type default))
+  )
+  (wire (pts (xy 193.04 59.69) (xy 200.66 59.69))
+    (stroke (width 0) (type default))
+  )
+  (wire (pts (xy 92.71 96.52) (xy 104.14 96.52))
+    (stroke (width 0) (type default))
+  )
+  (wire (pts (xy 137.16 157.48) (xy 137.16 152.4))
+    (stroke (width 0) (type default))
+  )
+  (wire (pts (xy 24.13 77.47) (xy 24.13 83.82))
+    (stroke (width 0) (type default))
+  )
   (wire (pts (xy 105.41 157.48) (xy 118.11 157.48))
     (stroke (width 0) (type default))
   )
-  (wire (pts (xy 92.71 92.71) (xy 92.71 96.52))
-    (stroke (width 0) (type default))
-  )
-  (wire (pts (xy 125.73 157.48) (xy 137.16 157.48))
-    (stroke (width 0) (type default))
-  )
-  (wire (pts (xy 118.11 101.6) (xy 118.11 110.49))
-    (stroke (width 0) (type default))
-  )
-  (wire (pts (xy 236.22 49.53) (xy 236.22 54.61))
-    (stroke (width 0) (type default))
-  )
-  (wire (pts (xy 193.04 49.53) (xy 236.22 49.53))
-    (stroke (width 0) (type default))
-  )
-  (wire (pts (xy 193.04 59.69) (xy 200.66 59.69))
-    (stroke (width 0) (type default))
-  )
-  (wire (pts (xy 92.71 96.52) (xy 104.14 96.52))
-    (stroke (width 0) (type default))
-  )
-  (wire (pts (xy 137.16 157.48) (xy 137.16 152.4))
-    (stroke (width 0) (type default))
-  )
-  (wire (pts (xy 24.13 77.47) (xy 24.13 83.82))
-    (stroke (width 0) (type default))
-  )
   (wire (pts (xy 73.66 157.48) (xy 73.66 158.75))
     (stroke (width 0) (type default))
@@
     (stroke (width 0) (type default))
   )
+  (bus (pts (xy 208.28 139.7) (xy 219.71 139.7))
+    (stroke (width 0) (type default))
+  )
   (wire (pts (xy 73.66 101.6) (xy 73.66 110.49))
     (stroke (width 0) (type default))
@@
     (stroke (width 0) (type default))
   )
-  (wire (pts (xy 118.11 157.48) (xy 119.38 157.48))
-    (stroke (width 0) (type default))
-  )
   (wire (pts (xy 193.04 57.15) (xy 200.66 57.15))
     (stroke (width 0) (type default))
@@
     (fill (type none))
   )
+  (rectangle (start 191.77 133.35) (end 236.22 149.86)
+    (stroke (width 0) (type default))
+    (fill (type none))
+  )
   (rectangle (start 20.32 68.58) (end 49.53 120.65)
     (stroke (width 0) (type default))
     (fill (type none))
+  )
+  (text "GLOBAL LABELS" (at 191.77 132.08 0)
+    (effects (font (size 1.27 1.27) bold) (justify left bottom))
   )
   (text "Power Supply, 3.3V" (at 67.31 66.04 0)
@@
     )
   )
+  (global_label "PWRU_IN" (shape input) (at 208.28 144.78 180) (fields_autoplaced)
+    (effects (font (size 1.27 1.27) bold) (justify right))
+    (property "Intersheetrefs" "${INTERSHEET_REFS}" (at 196.594 144.78 0)
+      (effects (font (size 1.27 1.27)) (justify right) hide)
+    )
+  )
   (global_label "PWRU_IN" (shape output) (at 59.69 149.86 0) (fields_autoplaced)
     (effects (font (size 1.27 1.27) bold) (justify left))
@@
     )
   )
+  (global_label "USBC_D{N,P}" (shape input) (at 208.28 139.7 180) (fields_autoplaced)
+    (effects (font (size 1.27 1.27) (thickness 0.254) bold) (justify right))
+    (property "Intersheetrefs" "${INTERSHEET_REFS}" (at 192.6025 139.7 0)
+      (effects (font (size 1.27 1.27)) (justify right) hide)
+    )
+  )
+  (hierarchical_label "PWRU_IN" (shape input) (at 220.98 144.78 0) (fields_autoplaced)
+    (effects (font (size 1.27 1.27) bold) (justify left))
+  )
+  (hierarchical_label "USBC_D{N,P}" (shape input) (at 219.71 139.7 0) (fields_autoplaced)
+    (effects (font (size 1.27 1.27)) (justify left))
+  )
   (symbol (lib_id "Device:C_Polarized_US") (at 118.11 97.79 0) (unit 1)
     (in_bom yes) (on_board yes) (dnp no)
@@
       (effects (font (size 1.27 1.27)))
     )
-    (property "Value" "FerriteBead" (at 83.7692 152.4 90)
+    (property "Value" "120" (at 83.7692 152.4 90)
       (effects (font (size 1.27 1.27)))
     )
@@
       (effects (font (size 1.27 1.27)) (justify left))
     )
-    (property "Value" "R" (at 232.41 59.69 0)
+    (property "Value" "5100" (at 232.41 59.69 0)
       (effects (font (size 1.27 1.27)) (justify left))
     )
@@
       (effects (font (size 1.27 1.27)) (justify left))
     )
-    (property "Value" "R" (at 44.45 91.44 0)
+    (property "Value" "70" (at 44.45 91.44 0)
       (effects (font (size 1.27 1.27)) (justify left))
     )
@@
       (effects (font (size 1.27 1.27)) (justify left))
     )
-    (property "Value" "R" (at 238.76 59.69 0)
+    (property "Value" "5.1k" (at 238.76 59.69 0)
       (effects (font (size 1.27 1.27)) (justify left))
     )
@@
       (effects (font (size 1.27 1.27)) (justify left))
     )
-    (property "Value" "C" (at 77.47 163.83 0)
+    (property "Value" ".01u" (at 77.47 163.83 0)
       (effects (font (size 1.27 1.27)) (justify left))
     )
@@
       (effects (font (size 1.27 1.27)))
     )
-    (property "Value" "Polyfuse" (at 121.92 153.67 90)
+    (property "Value" "500mA" (at 121.92 153.67 90)
       (effects (font (size 1.27 1.27)))
     )
@@
   (symbol (lib_id "Device:C_Polarized") (at 105.41 162.56 0) (unit 1)
     (in_bom yes) (on_board yes) (dnp no) (fields_autoplaced)
-    (property "Reference" "C11" (at 109.22 160.401 0)
-      (effects (font (size 1.27 1.27)) (justify left))
-    )
-    (property "Value" "C_Polarized" (at 109.22 162.941 0)
+    (property "Reference" "C15" (at 109.22 160.401 0)
+      (effects (font (size 1.27 1.27)) (justify left))
+    )
+    (property "Value" "4.7u" (at 109.22 162.941 0)
       (effects (font (size 1.27 1.27)) (justify left))
     )
@@
       (project "intro_to_pcb"
         (path "/b2bbdadf-112f-4546-9689-8793d1774710/fe0ea4a4-c2df-4c35-8e09-ee6e8be7cc0a"
-          (reference "C11") (unit 1)
+          (reference "C15") (unit 1)
         )
       )
@@
       (effects (font (size 1.27 1.27)) (justify left))
     )
-    (property "Value" "C" (at 93.98 163.83 0)
+    (property "Value" ".1u" (at 93.98 163.83 0)
       (effects (font (size 1.27 1.27)) (justify left))
     )
@@
       (effects (font (size 1.27 1.27)) (justify left))
     )
-    (property "Value" "R" (at 26.67 88.9 0)
-      (effects (font (size 1.27 1.27)) (justify left))
-    )
+    (property "Value" "155" (at 26.67 88.9 0)
+      (effects (font (size 1.27 1.27)) (justify left))
+    )

Commit message: updated
Parts:
- C10, C15, C7, C9: footprint (none) -> Capacitor_SMD:C_0603_1608Metric
- C8: footprint (none) -> Capacitor_SMD:C_0402_1005Metric
- D3, D4: footprint (none) -> LED_SMD:LED_0402_1005Metric
- F1: footprint (none) -> Fuse:Fuse_1812_4532Metric
- FB1: footprint (none) -> Resistor_SMD:R_0603_1608Metric
- J1: footprint (none) -> Connector_USB:USB_C_Receptacle_Palconn_UTC16-G
- R10, R5, R6, R7, R8, R9: footprint (none) -> Resistor_SMD:R_0402_1005Metric
- U2: footprint Package_TO_SOT_SMD:TO-252-3_TabPin2 -> Package_TO_SOT_SMD:SOT-223
Connections:
- net PWRU_IN: now also C9.1, FB1.1
Changed lines of the file:
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@@
-    (stroke (width 0) (type default))
-  )
-  (bus (pts (xy 208.28 144.78) (xy 220.98 144.78))
     (stroke (width 0) (type default))
   )
@@
     (stroke (width 0) (type default))
   )
+  (bus (pts (xy 208.28 139.7) (xy 219.71 139.7))
+    (stroke (width 0) (type default))
+  )
   (wire (pts (xy 118.11 110.49) (xy 104.14 110.49))
     (stroke (width 0) (type default))
@@
     (stroke (width 0) (type default))
   )
+  (wire (pts (xy 208.28 144.78) (xy 220.98 144.78))
+    (stroke (width 0) (type default))
+  )
   (wire (pts (xy 73.66 93.98) (xy 81.28 93.98))
     (stroke (width 0) (type default))
   )
   (wire (pts (xy 90.17 166.37) (xy 90.17 171.45))
-    (stroke (width 0) (type default))
-  )
-  (bus (pts (xy 208.28 139.7) (xy 219.71 139.7))
     (stroke (width 0) (type default))
   )
@@
     )
   )
-  (global_label "PWRU_IN" (shape output) (at 59.69 149.86 0) (fields_autoplaced)
-    (effects (font (size 1.27 1.27) bold) (justify left))
-    (property "Intersheetrefs" "${INTERSHEET_REFS}" (at 71.376 149.86 0)
-      (effects (font (size 1.27 1.27)) (justify left) hide)
+  (global_label "PWRU_IN" (shape input) (at 69.85 149.86 180) (fields_autoplaced)
+    (effects (font (size 1.27 1.27) bold) (justify right))
+    (property "Intersheetrefs" "${INTERSHEET_REFS}" (at 58.164 149.86 0)
+      (effects (font (size 1.27 1.27)) (justify right) hide)
     )
   )
@@
       (effects (font (size 1.27 1.27)) (justify left))
     )
-    (property "Footprint" "" (at 118.11 97.79 0)
+    (property "Footprint" "Capacitor_SMD:C_0402_1005Metric" (at 118.11 97.79 0)
       (effects (font (size 1.27 1.27)) hide)
     )
@@
       (effects (font (size 1.27 1.27)) (justify right))
     )
-    (property "Footprint" "" (at 24.13 101.6 0)
+    (property "Footprint" "LED_SMD:LED_0402_1005Metric" (at 24.13 101.6 0)
       (effects (font (size 1.27 1.27)) hide)
     )
@@
       (effects (font (size 1.27 1.27)))
     )
-    (property "Footprint" "" (at 83.82 159.258 90)
+    (property "Footprint" "Resistor_SMD:R_0603_1608Metric" (at 83.82 159.258 90)
       (effects (font (size 1.27 1.27)) hide)
     )
@@
       (effects (font (size 1.27 1.27)) (justify left))
     )
-    (property "Footprint" "" (at 228.092 58.42 90)
+    (property "Footprint" "Resistor_SMD:R_0402_1005Metric" (at 228.092 58.42 90)
       (effects (font (size 1.27 1.27)) hide)
     )
@@
       (effects (font (size 1.27 1.27)) (justify left))
     )
-    (property "Footprint" "" (at 40.132 90.17 90)
+    (property "Footprint" "Resistor_SMD:R_0402_1005Metric" (at 40.132 90.17 90)
       (effects (font (size 1.27 1.27)) hide)
     )
@@
       (effects (font (size 1.27 1.27)) (justify left))
     )
-    (property "Footprint" "" (at 234.442 58.42 90)
+    (property "Footprint" "Resistor_SMD:R_0402_1005Metric" (at 234.442 58.42 90)
       (effects (font (size 1.27 1.27)) hide)
     )
@@
       (effects (font (size 1.27 1.27)))
     )
-    (property "Footprint" "" (at 181.61 59.69 0)
+    (property "Footprint" "Connector_USB:USB_C_Receptacle_Palconn_UTC16-G" (at 181.61 59.69 0)
       (effects (font (size 1.27 1.27)) hide)
     )
@@
       (effects (font (size 1.27 1.27)) (justify right))
     )
-    (property "Footprint" "" (at 41.91 102.87 0)
+    (property "Footprint" "LED_SMD:LED_0402_1005Metric" (at 41.91 102.87 0)
       (effects (font (size 1.27 1.27)) hide)
     )
@@
       (effects (font (size 1.27 1.27)) (justify left))
     )
-    (property "Footprint" "" (at 74.6252 166.37 0)
+    (property "Footprint" "Capacitor_SMD:C_0603_1608Metric" (at 74.6252 166.37 0)
       (effects (font (size 1.27 1.27)) hide)
     )
@@
       (effects (font (size 1.27 1.27)))
     )
-    (property "Footprint" "Package_TO_SOT_SMD:TO-252-3_TabPin2" (at 92.71 85.09 0)
+    (property "Footprint" "Package_TO_SOT_SMD:SOT-223" (at 92.71 85.09 0)
       (effects (font (size 1.27 1.27)) hide)
     )
@@
       (effects (font (size 1.27 1.27)))
     )
-    (property "Footprint" "" (at 127 156.21 0)
+    (property "Footprint" "Fuse:Fuse_1812_4532Metric" (at 127 156.21 0)
       (effects (font (size 1.27 1.27)) (justify left) hide)
     )
@@
       (effects (font (size 1.27 1.27)) (justify left))
     )
-    (property "Footprint" "" (at 102.362 102.87 90)
+    (property "Footprint" "Resistor_SMD:R_0402_1005Metric" (at 102.362 102.87 90)
       (effects (font (size 1.27 1.27)) hide)
     )
@@
       (effects (font (size 1.27 1.27)) (justify left))
     )
-    (property "Footprint" "" (at 106.3752 166.37 0)
+    (property "Footprint" "Capacitor_SMD:C_0603_1608Metric" (at 106.3752 166.37 0)
       (effects (font (size 1.27 1.27)) hide)
     )
@@
       (effects (font (size 1.27 1.27)) (justify left))
     )
-    (property "Footprint" "" (at 73.66 97.79 0)
+    (property "Footprint" "Capacitor_SMD:C_0603_1608Metric" (at 73.66 97.79 0)
       (effects (font (size 1.27 1.27)) hide)
     )
@@
       (effects (font (size 1.27 1.27)) (justify left))
     )
-    (property "Footprint" "" (at 91.1352 166.37 0)
+    (property "Footprint" "Capacitor_SMD:C_0603_1608Metric" (at 91.1352 166.37 0)
       (effects (font (size 1.27 1.27)) hide)
     )
@@
       (effects (font (size 1.27 1.27)) (justify left))
     )
-    (property "Footprint" "" (at 102.362 91.44 90)
+    (property "Footprint" "Resistor_SMD:R_0402_1005Metric" (at 102.362 91.44 90)
       (effects (font (size 1.27 1.27)) hide)
     )
@@
       (effects (font (size 1.27 1.27)) (justify left))
     )
-    (property "Footprint" "" (at 22.352 87.63 90)
-      (effects (font (size 1.27 1.27)) hide)
-    )
+    (property "Footprint" "Resistor_SMD:R_0402_1005Metric" (at 22.352 87.63 90)
+      (effects (font (size 1.27 1.27)) hide)
+    )
