File: intro_to_pcb.kicad_pcb (KiCad board)
At the start: 2 copper layers, 0 parts

Commit message: updated
Parts:
- added C1: .1u, Capacitor_SMD:C_0402_1005Metric, F.Cu at (153.1, 99.7)
- added C10: .1u, Capacitor_SMD:C_0603_1608Metric, F.Cu at (156.6, 76.5)
- added C11: .1u, Capacitor_SMD:C_0603_1608Metric, F.Cu at (147.7, 112.0)
- added C12: .1u, Capacitor_SMD:C_0402_1005Metric, F.Cu at (147.2, 103.7)
- added C13: 4.7u, Capacitor_SMD:C_0402_1005Metric, F.Cu at (147.2, 105.6)
- added C14: C_Polarized, Capacitor_SMD:CP_Elec_6.3x7.7, F.Cu at (140.4, 114.8)
- added C15: 4.7u, Capacitor_SMD:C_0603_1608Metric, F.Cu at (156.6, 79.0)
- added C2: .1u, Capacitor_SMD:C_0402_1005Metric, F.Cu at (153.1, 101.6)
- added C3: 18p, Capacitor_SMD:C_0402_1005Metric, F.Cu at (153.1, 103.6)
- added C4: 18p, Capacitor_SMD:C_0402_1005Metric, F.Cu at (153.1, 105.6)
- added C5: .1u, Capacitor_SMD:C_0402_1005Metric, F.Cu at (153.1, 107.5)
- added C6: .1u, Capacitor_SMD:C_0402_1005Metric, F.Cu at (153.1, 109.5)
- added C7: 10u, Capacitor_SMD:C_0603_1608Metric, F.Cu at (156.6, 71.5)
- added C8: 10u, Capacitor_SMD:C_0402_1005Metric, F.Cu at (171.7, 80.8)
- added C9: .01u, Capacitor_SMD:C_0603_1608Metric, F.Cu at (156.6, 74.0)
- added D1: 1.5KExxCA, Diode_THT:D_DO-201AE_P15.24mm_Horizontal, F.Cu at (137.3, 73.7)
- added D2: 1.5KExxCA, Diode_THT:D_DO-201AE_P15.24mm_Horizontal, F.Cu at (137.3, 80.5)
- added D3: LED, LED_SMD:LED_0402_1005Metric, F.Cu at (194.2, 78.8)
- added D4: LED, LED_SMD:LED_0402_1005Metric, F.Cu at (194.2, 80.8)
- added D5: TX_LED, LED_SMD:LED_0402_1005Metric, F.Cu at (147.5, 99.7)
- added F1: 500mA, Fuse:Fuse_1812_4532Metric, F.Cu at (189.1, 80.3)
- added FB1: 120, Resistor_SMD:R_0603_1608Metric, F.Cu at (156.6, 81.5)
- added J1: USB_C_Receptacle_USB2.0_16P, Connector_USB:USB_C_Receptacle_Palconn_UTC16-G, F.Cu at (176.0, 74.0)
- added J2: Conn_01x16_Socket, Connector_PinHeader_2.54mm:PinHeader_1x16_P2.54mm_Vertical, F.Cu at (119.1, 72.1)
- added J3: Conn_01x16_Socket, Connector_PinHeader_2.54mm:PinHeader_1x16_P2.54mm_Vertical, F.Cu at (123.8, 72.1)
- added J4: Conn_PIC_ICSP_ICD, Connector_PinSocket_2.54mm:PinSocket_2x03_P2.54mm_Vertical, F.Cu at (130.9, 72.1)
- added L1: 10u, Inductor_SMD:L_0603_1608Metric, F.Cu at (163.1, 111.6)
- added R1: R, Resistor_SMD:R_0402_1005Metric, F.Cu at (167.7, 99.7)
- added R10: 70, Resistor_SMD:R_0402_1005Metric, F.Cu at (168.8, 80.8)
- added R11: 150, Resistor_SMD:R_0402_1005Metric, F.Cu at (147.1, 114.2)
- added R12: 150, Resistor_SMD:R_0402_1005Metric, F.Cu at (147.1, 116.2)
- added R2: R, Resistor_SMD:R_0402_1005Metric, F.Cu at (167.7, 101.7)
- added R3: R, Resistor_SMD:R_0402_1005Metric, F.Cu at (167.7, 103.7)
- added R4: 10k, Resistor_SMD:R_0402_1005Metric, F.Cu at (167.7, 105.7)
- added R5: 121, Resistor_SMD:R_0402_1005Metric, F.Cu at (168.8, 70.8)
- added R6: 200, Resistor_SMD:R_0402_1005Metric, F.Cu at (168.8, 72.8)
- added R7: 5100, Resistor_SMD:R_0402_1005Metric, F.Cu at (168.8, 74.8)
- added R8: 5.1k, Resistor_SMD:R_0402_1005Metric, F.Cu at (168.8, 76.8)
- added R9: 155, Resistor_SMD:R_0402_1005Metric, F.Cu at (168.8, 78.8)
- added RX_LED1: LED, LED_SMD:LED_0402_1005Metric, F.Cu at (147.5, 101.7)
- added SW1: SW_Push, Button_Switch_SMD:SW_Push_SPST_NO_Alps_SKRK, F.Cu at (157.8, 112.6)
- added U1: ATmega328P-A, Package_QFP:TQFP-32_7x7mm_P0.8mm, F.Cu at (160.4, 104.5)
- added U2: LM1117DT-ADJ, Package_TO_SOT_SMD:SOT-223, F.Cu at (190.5, 73.7)
- added U3: FT232RL, Package_SO:SSOP-28_5.3x10.2mm_P0.65mm, F.Cu at (140.5, 104.7)
- added Y1: 16Mhz, Crystal:Crystal_SMD_2012-2Pin_2.0x1.2mm, F.Cu at (166.9, 111.8)
