File: untitled.kicad_sch (KiCad schematic)
At the start: 9 parts, among them U3 FT232RL

Commit message: updated
Parts:
- C11: footprint (none) -> Capacitor_SMD:C_0603_1608Metric
- C12, C13: footprint (none) -> Capacitor_SMD:C_0402_1005Metric
- C14: footprint (none) -> Capacitor_SMD:CP_Elec_6.3x7.7
- D5, RX_LED1: footprint (none) -> LED_SMD:LED_0402_1005Metric
- R11, R12: footprint (none) -> Resistor_SMD:R_0402_1005Metric
Connections:
- net EX_RST: now also C14.2
- net GND: now also U3.25 (AGND)
- net USART_DTR: now also C14.1
- net USB_D.N: now also U3.16 (USBD-)
- net USB_D.P: now also U3.15 (USBD+)
Changed lines of the file:
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@@
   (junction (at 256.54 68.58) (diameter 0) (color 0 0 0 0)
+  )
+  (junction (at 137.16 119.38) (diameter 0) (color 0 0 0 0)
   )
   (junction (at 194.31 96.52) (diameter 0) (color 0 0 0 0)
@@
     (stroke (width 0) (type default))
   )
+  (wire (pts (xy 157.48 96.52) (xy 160.02 96.52))
+    (stroke (width 0) (type default))
+  )
+  (wire (pts (xy 137.16 57.15) (xy 139.7 57.15))
+    (stroke (width 0) (type default))
+  )
+  (wire (pts (xy 157.48 81.28) (xy 163.83 81.28))
+    (stroke (width 0) (type default))
+  )
   (bus (pts (xy 74.93 165.1) (xy 80.01 165.1))
     (stroke (width 0) (type default))
   )
-  (wire (pts (xy 157.48 96.52) (xy 160.02 96.52))
-    (stroke (width 0) (type default))
-  )
-  (wire (pts (xy 137.16 57.15) (xy 139.7 57.15))
-    (stroke (width 0) (type default))
-  )
-  (wire (pts (xy 157.48 81.28) (xy 163.83 81.28))
-    (stroke (width 0) (type default))
-  )
   (wire (pts (xy 139.7 119.38) (xy 139.7 120.65))
     (stroke (width 0) (type default))
@@
     (stroke (width 0) (type default))
   )
+  (bus (pts (xy 71.12 160.02) (xy 82.55 160.02))
+    (stroke (width 0) (type default))
+  )
   (wire (pts (xy 186.69 99.06) (xy 194.31 99.06))
     (stroke (width 0) (type default))
@@
     (stroke (width 0) (type default))
   )
-  (bus (pts (xy 71.12 160.02) (xy 82.55 160.02))
+  (wire (pts (xy 137.16 119.38) (xy 139.7 119.38))
     (stroke (width 0) (type default))
   )
@@
     (stroke (width 0) (type default))
   )
-  (wire (pts (xy 137.16 119.38) (xy 139.7 119.38))
+  (wire (pts (xy 132.08 119.38) (xy 137.16 119.38))
     (stroke (width 0) (type default))
   )
   (wire (pts (xy 194.31 96.52) (xy 194.31 99.06))
+    (stroke (width 0) (type default))
+  )
+  (wire (pts (xy 132.08 114.3) (xy 132.08 119.38))
     (stroke (width 0) (type default))
   )
@@
     (effects (font (size 1.27 1.27) bold) (justify left bottom))
   )
-  (global_label "USB_D.P" (shape output) (at 99.06 78.74 0) (fields_autoplaced)
-    (effects (font (size 1.27 1.27)) (justify left))
-    (property "Intersheetrefs" "${INTERSHEET_REFS}" (at 109.9676 78.74 0)
-      (effects (font (size 1.27 1.27)) (justify left) hide)
+  (global_label "USB_D.P" (shape input) (at 109.22 78.74 180) (fields_autoplaced)
+    (effects (font (size 1.27 1.27)) (justify right))
+    (property "Intersheetrefs" "${INTERSHEET_REFS}" (at 98.3124 78.74 0)
+      (effects (font (size 1.27 1.27)) (justify right) hide)
     )
   )
@@
     )
   )
-  (global_label "EX_RST" (shape output) (at 234.95 105.41 0) (fields_autoplaced)
-    (effects (font (size 1.27 1.27) (thickness 0.254) bold) (justify left))
-    (property "Intersheetrefs" "${INTERSHEET_REFS}" (at 245.1844 105.41 0)
-      (effects (font (size 1.27 1.27)) (justify left) hide)
-    )
-  )
-  (global_label "USB_D.N" (shape output) (at 99.06 81.28 0) (fields_autoplaced)
-    (effects (font (size 1.27 1.27)) (justify left))
-    (property "Intersheetrefs" "${INTERSHEET_REFS}" (at 110.0281 81.28 0)
-      (effects (font (size 1.27 1.27)) (justify left) hide)
+  (global_label "EX_RST" (shape input) (at 243.84 105.41 180) (fields_autoplaced)
+    (effects (font (size 1.27 1.27) (thickness 0.254) bold) (justify right))
+    (property "Intersheetrefs" "${INTERSHEET_REFS}" (at 233.6056 105.41 0)
+      (effects (font (size 1.27 1.27)) (justify right) hide)
+    )
+  )
+  (global_label "USB_D.N" (shape input) (at 109.22 81.28 180) (fields_autoplaced)
+    (effects (font (size 1.27 1.27)) (justify right))
+    (property "Intersheetrefs" "${INTERSHEET_REFS}" (at 98.2519 81.28 0)
+      (effects (font (size 1.27 1.27)) (justify right) hide)
     )
   )
@@
     )
   )
-  (global_label "USART_DTR" (shape output) (at 233.68 95.25 0) (fields_autoplaced)
-    (effects (font (size 1.27 1.27)) (justify left))
-    (property "Intersheetrefs" "${INTERSHEET_REFS}" (at 247.0066 95.25 0)
-      (effects (font (size 1.27 1.27)) (justify left) hide)
+  (global_label "USART_DTR" (shape input) (at 246.38 95.25 180) (fields_autoplaced)
+    (effects (font (size 1.27 1.27)) (justify right))
+    (property "Intersheetrefs" "${INTERSHEET_REFS}" (at 233.0534 95.25 0)
+      (effects (font (size 1.27 1.27)) (justify right) hide)
     )
   )
@@
       (effects (font (size 1.27 1.27)) (justify left))
     )
-    (property "Footprint" "" (at 82.2452 81.28 0)
+    (property "Footprint" "Capacitor_SMD:C_0603_1608Metric" (at 82.2452 81.28 0)
       (effects (font (size 1.27 1.27)) hide)
     )
@@
       (effects (font (size 1.27 1.27)) (justify left))
     )
-    (property "Footprint" "" (at 257.5052 63.5 0)
+    (property "Footprint" "Capacitor_SMD:C_0402_1005Metric" (at 257.5052 63.5 0)
       (effects (font (size 1.27 1.27)) hide)
     )
@@
       (effects (font (size 1.27 1.27)))
     )
-    (property "Footprint" "" (at 163.83 96.52 0)
+    (property "Footprint" "LED_SMD:LED_0402_1005Metric" (at 163.83 96.52 0)
       (effects (font (size 1.27 1.27)) hide)
     )
@@
       (effects (font (size 1.27 1.27)))
     )
-    (property "Footprint" "" (at 172.72 99.06 0)
+    (property "Footprint" "LED_SMD:LED_0402_1005Metric" (at 172.72 99.06 0)
       (effects (font (size 1.27 1.27)) hide)
     )
@@
       (effects (font (size 1.27 1.27)) (justify left))
     )
-    (property "Footprint" "" (at 258.7752 102.87 0)
+    (property "Footprint" "Capacitor_SMD:CP_Elec_6.3x7.7" (at 258.7752 102.87 0)
       (effects (font (size 1.27 1.27)) hide)
     )
@@
       (effects (font (size 1.27 1.27)))
     )
-    (property "Footprint" "" (at 182.88 97.282 90)
+    (property "Footprint" "Resistor_SMD:R_0402_1005Metric" (at 182.88 97.282 90)
       (effects (font (size 1.27 1.27)) hide)
     )
@@
       (effects (font (size 1.27 1.27)) (justify left))
     )
-    (property "Footprint" "" (at 239.7252 63.5 0)
+    (property "Footprint" "Capacitor_SMD:C_0402_1005Metric" (at 239.7252 63.5 0)
       (effects (font (size 1.27 1.27)) hide)
     )
@@
       (effects (font (size 1.27 1.27)))
     )
-    (property "Footprint" "" (at 173.99 94.742 90)
-      (effects (font (size 1.27 1.27)) hide)
-    )
+    (property "Footprint" "Resistor_SMD:R_0402_1005Metric" (at 173.99 94.742 90)
+      (effects (font (size 1.27 1.27)) hide)
+    )
